Commit message: update

File: my_robot/urdf/my.urdf (robot description, URDF)
Before this commit: robot my, 7 links, 6 joints
Links:
- added link camera_link, mass 0.05; collision box size=0.03 0.03 0.02; visual box size=0.03 0.03 0.02
- added link camera_link_optical
- link base_link: mass None -> 2.0; geometry collision cylinder length=0.05 radius=0.15; visual mesh filename=package://my_robot/meshes/base.STL scale=0.01 0.01 0.01
- link link0: mass None -> 0.8; geometry collision cylinder length=0.15 radius=0.08; visual mesh filename=package://my_robot/meshes/joint1.STL scale=0.01 0.01 0.01
- link link1: mass None -> 0.7; geometry collision box size=0.15 0.06 0.06; visual mesh filename=package://my_robot/meshes/joint2.STL scale=0.01 0.01 0.01
- link link2: mass None -> 0.6; geometry collision box size=0.15 0.06 0.06; visual mesh filename=package://my_robot/meshes/joint3.STL scale=0.01 0.01 0.01
- link link3: mass None -> 0.5; geometry collision box size=0.12 0.05 0.05; visual mesh filename=package://my_robot/meshes/joint4.STL scale=0.01 0.01 0.01
- link link4: mass None -> 0.4; geometry collision box size=0.10 0.04 0.04; visual mesh filename=package://my_robot/meshes/joint5.STL scale=0.01 0.01 0.01
- link link5: mass None -> 0.3; geometry collision cylinder length=0.06 radius=0.04
Joints:
- added joint camera_optical_joint: type fixed, parent camera_link, child camera_link_optical, origin xyz=0 0 0 rpy=0 0 3.1415
- added joint link5_to_camera: type fixed, parent link5, child camera_link, origin xyz=0.0 0.406 0.39 rpy=0 0 0
- joint link2_to_link3: origin xyz=0.0 0.7 0.0 rpy=-1.5708  0 1.5708 -> xyz=0.0 0.7 0.0 rpy=-1.5708 0 1.5708
